File: sch/rusty-hangulclock/rusty-hangulclock.kicad_pcb (KiCad board)
At the start: 2 copper layers, 53.5 x 54 mm, 13 parts, among them J1 Conn_OLED, J2 Conn_LEDS, J3 PWR, SW1 SW_Push

Commit message: sch: pcb round routes
Routing:
- net +5V: track 104.8 -> 102.6 mm
- net GND: track 128.1 -> 126.1 mm
- net +3V3: track 60.5 -> 59.5 mm
- net Net-(J2-Pin_4): track 42.9 -> 42.0 mm
- net Net-(J1-Pin_4): track 37.1 -> 36.2 mm
- net Net-(J1-Pin_5): track 32.4 -> 31.6 mm
- net Net-(J1-Pin_3): track 41.7 -> 40.9 mm
- net Net-(J2-Pin_3): track 26.6 -> 26.0 mm
- net Net-(J2-Pin_5): track 27.1 -> 26.5 mm
- net Net-(M1-P1): track 27.9 -> 27.3 mm
