File: sch/rusty-hangulclock/rusty-hangulclock.kicad_pcb (KiCad board)
At the start: 2 copper layers, 45 x 54 mm, 14 parts, among them J1 Conn_OLED, J2 Conn_SLEDS, J3 PWR, SW1 RotaryEncoder_Switch_MP

Commit message: feat: rev7.
Parts:
- added U1: 74AHCT125, Package_SO:SOIC-14_3.9x8.7mm_P1.27mm, B.Cu at (130.5, 101.0)
- moved C4 25.6 mm to (159.0, 98.5), turned to 90 degrees
- moved C3 5.00 mm to (135.2, 89.0)
- moved C2 4.75 mm to (135.2, 94.0)
Connections:
- J2 pad 2: GND -> Net-(J2-Pin_2)
- J2 pad 3: Net-(ESP32-C3_SuperMini1-P6) -> Net-(J2-Pin_3)
- J2 pad 4: Net-(ESP32-C3_SuperMini1-P4) -> GND
Routing:
- net +5V: track 27.0 -> 58.4 mm
- net Net-(J2-Pin_3): track 0.00 -> 11.8 mm
- net Net-(J2-Pin_2): track 0.00 -> 11.6 mm
- net Net-(ESP32-C3_SuperMini1-P3): track 60.9 -> 49.9 mm
- net Net-(ESP32-C3_SuperMini1-P6): track 38.7 -> 45.0 mm
- net Net-(ESP32-C3_SuperMini1-P1): track 31.7 -> 36.5 mm
- net Net-(ESP32-C3_SuperMini1-P2): track 41.0 -> 45.8 mm
- net Net-(ESP32-C3_SuperMini1-P4): track 28.6 -> 32.2 mm, vias 0 -> 1
- net GND: vias 1 -> 4
Other:
- board text added: "Rusty HangulClock By Homin Lee May 2025 https://github.com/suapapa /rusty-hangulclock"
- board text removed: "Rusty HangulClock By Homin Lee Feb 2025 https://github.com/ suapapa/HangulClock"
